File: xns-ip67.sch (EAGLE design)
At the start: 119 parts, among them J1 DCJ0202

Commit message: Rev 0
First Version without routing
Parts:
- removed SV1: (no value), con-lstb:MA03-1
- added 5.5V, PAD115, PAD116: WIREPAD1,6/0,9, wirepad:WIREPAD1,6/0,9
- added JP1, JP10, JP11, JP12, JP13, JP14, JP15, JP16, JP17, JP18, JP19, JP2, JP20, JP21, JP22, JP23, JP24, JP25, JP26, JP27, JP28, JP29, JP3, JP30, JP35, JP36, JP4, JP5, JP6, JP7, JP8, JP9: (no value), adafruit:PINHD-1X8CLEANBIG
- added JP31, JP32, JP33, JP34: (no value), microbuilder:HEADER-1X12
- added PROG: (no value), con-lstb:MA03-1
- added U1: (no value), SparkFun-PowerIC:MIC52053.3V
- added X2: (no value), microbuilder:USBMICRO_20329
Connections:
- new net N$23: JP3.1, JP3.2, JP3.3, JP3.4, JP3.5, JP3.6, JP3.7, JP3.8
- new net N$24: JP4.1, JP4.2, JP4.3, JP4.4, JP4.5, JP4.6, JP4.7, JP4.8
- new net N$25: JP5.1, JP5.2, JP5.3, JP5.4, JP5.5, JP5.6, JP5.7, JP5.8
- new net N$26: JP6.1, JP6.2, JP6.3, JP6.4, JP6.5, JP6.6, JP6.7, JP6.8
- new net N$27: JP7.1, JP7.2, JP7.3, JP7.4, JP7.5, JP7.6, JP7.7, JP7.8
- new net N$28: JP8.1, JP8.2, JP8.3, JP8.4, JP8.5, JP8.6, JP8.7, JP8.8
- new net N$29: JP9.1, JP9.2, JP9.3, JP9.4, JP9.5, JP9.6, JP9.7, JP9.8
- new net N$30: JP10.1, JP10.2, JP10.3, JP10.4, JP10.5, JP10.6, JP10.7, JP10.8
- new net N$31: JP11.1, JP11.2, JP11.3, JP11.4, JP11.5, JP11.6, JP11.7, JP11.8
- new net N$32: JP12.1, JP12.2, JP12.3, JP12.4, JP12.5, JP12.6, JP12.7, JP12.8
- new net N$33: JP13.1, JP13.2, JP13.3, JP13.4, JP13.5, JP13.6, JP13.7, JP13.8
- new net N$34: JP14.1, JP14.2, JP14.3, JP14.4, JP14.5, JP14.6, JP14.7, JP14.8
- new net N$35: JP15.1, JP15.2, JP15.3, JP15.4, JP15.5, JP15.6, JP15.7, JP15.8
- new net N$36: JP30.1, JP30.2, JP30.3, JP30.4, JP30.5, JP30.6, JP30.7, JP30.8
- new net N$37: JP29.1, JP29.2, JP29.3, JP29.4, JP29.5, JP29.6, JP29.7, JP29.8
- new net N$38: JP28.1, JP28.2, JP28.3, JP28.4, JP28.5, JP28.6, JP28.7, JP28.8
- new net N$39: JP27.1, JP27.2, JP27.3, JP27.4, JP27.5, JP27.6, JP27.7, JP27.8
- new net N$40: JP26.1, JP26.2, JP26.3, JP26.4, JP26.5, JP26.6, JP26.7, JP26.8
- new net N$41: JP25.1, JP25.2, JP25.3, JP25.4, JP25.5, JP25.6, JP25.7, JP25.8
- new net N$42: JP24.1, JP24.2, JP24.3, JP24.4, JP24.5, JP24.6, JP24.7, JP24.8
- new net N$43: JP22.1, JP22.2, JP22.3, JP22.4, JP22.5, JP22.6, JP22.7, JP22.8
- new net N$44: JP21.1, JP21.2, JP21.3, JP21.4, JP21.5, JP21.6, JP21.7, JP21.8
- new net N$45: JP20.1, JP20.2, JP20.3, JP20.4, JP20.5, JP20.6, JP20.7, JP20.8
- new net N$46: JP19.1, JP19.2, JP19.3, JP19.4, JP19.5, JP19.6, JP19.7, JP19.8
- new net N$47: JP18.1, JP18.2, JP18.3, JP18.4, JP18.5, JP18.6, JP18.7, JP18.8
- new net N$48: JP17.1, JP17.2, JP17.3, JP17.4, JP17.5, JP17.6, JP17.7, JP17.8
- new net N$49: JP16.1, JP16.2, JP16.3, JP16.4, JP16.5, JP16.6, JP16.7, JP16.8
- new net N$50: JP35.1, JP35.2, JP35.3, JP35.4, JP35.5, JP35.6, JP35.7, JP35.8
- new net N$51: JP36.1, JP36.2, JP36.3, JP36.4, JP36.5, JP36.6, JP36.7, JP36.8
- net GND: now also JP31.1, JP31.10, JP31.11, JP31.12, JP31.2, JP31.3, JP31.4, JP31.5, JP31.6, JP31.7, JP31.8, JP31.9, JP32.1, JP32.10, JP32.11, JP32.12, JP32.2, JP32.3, JP32.4, JP32.5, JP32.6, JP32.7, JP32.8, JP32.9, MDL1.GND, PAD107.P, PAD108.P, PAD109.P, PAD110.P, PAD111.P, PAD25.P, PAD26.P, PAD39.P, PAD40.P, PROG.1, U1.GND, X1-2.KL, X2.GND
- net N$14: now also MDL1.SCLK
- net N$15: now also MDL1.GPIO15
- net N$16: now also MDL1.GPIO2
- net N$17: now also MDL1.GPIO0
- net N$18: now also MDL1.GPIO4
- net N$19: now also MDL1.GPIO5
- net N$20: now also MDL1.TXD, PROG.3; no longer PAD103.P, PAD104.P, PAD105.P, PAD106.P
- net N$21: now also JP1.1, JP1.2, JP1.3, JP1.4, JP1.5, JP1.6, JP1.7, JP1.8; no longer PAD107.P, PAD108.P, PAD109.P, PAD110.P
- net N$22: now also JP2.1, JP2.2, JP2.3, JP2.4, JP2.5, JP2.6, JP2.7, JP2.8; no longer PAD111.P, PAD112.P, PAD113.P, PAD114.P
- net N$4: now also MDL1.RXD, PROG.2; no longer MDL1.VCC, PAD39.P, PAD40.P, PAD41.P, PAD42.P
- net VCC: now also 5.5V.P, U1.EN, U1.IN, X1-1.KL, X2.VBUS
- net VDD: now also JP33.1, JP33.10, JP33.11, JP33.12, JP33.2, JP33.3, JP33.4, JP33.5, JP33.6, JP33.7, JP33.8, JP33.9, JP34.1, JP34.10, JP34.11, JP34.12, JP34.2, JP34.3, JP34.4, JP34.5, JP34.6, JP34.7, JP34.8, JP34.9, MDL1.VCC, PAD103.P, PAD104.P, PAD105.P, PAD106.P, PAD112.P, PAD113.P, PAD114.P, PAD115.P, PAD116.P, PAD41.P, PAD42.P, U1.OUT; no longer PAD25.P, PAD26.P
