File: xns-ip67.sch (EAGLE design)
At the start: 86 parts, among them J1 DCJ0202

Commit message: Version without esp8266
Simple version
Parts:
- removed PAD1, PAD10, PAD103, PAD104, PAD105, PAD106, PAD107, PAD108, PAD109, PAD11, PAD110, PAD111, PAD112, PAD113, PAD114, PAD115, PAD116, PAD12, PAD13, PAD14, PAD15, PAD16, PAD17, PAD18, PAD19, PAD2, PAD20, PAD21, PAD22, PAD23, PAD24, PAD25, PAD26, PAD3, PAD39, PAD4, PAD40, PAD41, PAD42, PAD5, PAD6, PAD7, PAD8, PAD9: WIREPAD1,6/0,9, wirepad:WIREPAD1,6/0,9
- removed X1: (no value), con-ptr500:AK300/2
- added J2, J3, J4, J5: (no value), SparkFun-Connectors:M111X11_NO_SILK
Connections:
- net GND: now also J2.1, J2.10, J2.11, J2.2, J2.3, J2.4, J2.5, J2.6, J2.7, J2.8, J2.9, J4.1, J4.10, J4.11, J4.2, J4.3, J4.4, J4.5, J4.6, J4.7, J4.8, J4.9; no longer PAD1.P, PAD107.P, PAD108.P, PAD109.P, PAD110.P, PAD111.P, PAD13.P, PAD14.P, PAD15.P, PAD16.P, PAD17.P, PAD18.P, PAD19.P, PAD2.P, PAD25.P, PAD26.P, PAD3.P, PAD39.P, PAD4.P, PAD40.P, PAD5.P, PAD6.P, X1-2.KL
- net VCC: no longer X1-1.KL
- net VDD: now also J3.1, J3.10, J3.11, J3.2, J3.3, J3.4, J3.5, J3.6, J3.7, J3.8, J3.9, J5.1, J5.10, J5.11, J5.2, J5.3, J5.4, J5.5, J5.6, J5.7, J5.8, J5.9; no longer PAD10.P, PAD103.P, PAD104.P, PAD105.P, PAD106.P, PAD11.P, PAD112.P, PAD113.P, PAD114.P, PAD115.P, PAD116.P, PAD12.P, PAD20.P, PAD21.P, PAD22.P, PAD23.P, PAD24.P, PAD41.P, PAD42.P, PAD7.P, PAD8.P, PAD9.P

Commit message: Routed and Gerb files
Routed and produced verb files
Parts:
- added J10, J11, J12, J13, J14, J15, J16, J17, J18, J19, J20, J21, J22, J23, J24, J25, J26, J27, J6, J7, J8, J9: (no value), SparkFun-Connectors:M09NO_SILK
Connections:
- new net N$1: J6.1, J6.2, J6.3, J6.4, J6.5, J6.6, J6.7, J6.8, J6.9
- new net N$10: J15.1, J15.2, J15.3, J15.4, J15.5, J15.6, J15.7, J15.8, J15.9
- new net N$11: J16.1, J16.2, J16.3, J16.4, J16.5, J16.6, J16.7, J16.8, J16.9
- new net N$12: J17.1, J17.2, J17.3, J17.4, J17.5, J17.6, J17.7, J17.8, J17.9
- new net N$13: J18.1, J18.2, J18.3, J18.4, J18.5, J18.6, J18.7, J18.8, J18.9
- new net N$14: J19.1, J19.2, J19.3, J19.4, J19.5, J19.6, J19.7, J19.8, J19.9
- new net N$15: J20.1, J20.2, J20.3, J20.4, J20.5, J20.6, J20.7, J20.8, J20.9
- new net N$16: J21.1, J21.2, J21.3, J21.4, J21.5, J21.6, J21.7, J21.8, J21.9
- new net N$17: J22.1, J22.2, J22.3, J22.4, J22.5, J22.6, J22.7, J22.8, J22.9
- new net N$18: J23.1, J23.2, J23.3, J23.4, J23.5, J23.6, J23.7, J23.8, J23.9
- new net N$19: J24.1, J24.2, J24.3, J24.4, J24.5, J24.6, J24.7, J24.8, J24.9
- new net N$2: J7.1, J7.2, J7.3, J7.4, J7.5, J7.6, J7.7, J7.8, J7.9
- new net N$20: J25.1, J25.2, J25.3, J25.4, J25.5, J25.6, J25.7, J25.8, J25.9
- new net N$3: J8.1, J8.2, J8.3, J8.4, J8.5, J8.6, J8.7, J8.8, J8.9
- new net N$4: J9.1, J9.2, J9.3, J9.4, J9.5, J9.6, J9.7, J9.8, J9.9
- new net N$5: J10.1, J10.2, J10.3, J10.4, J10.5, J10.6, J10.7, J10.8, J10.9
- new net N$52: J26.1, J26.2, J26.3, J26.4, J26.5, J26.6, J26.7, J26.8, J26.9
- new net N$53: J27.1, J27.2, J27.3, J27.4, J27.5, J27.6, J27.7, J27.8, J27.9
- new net N$54: JP23.1, JP23.2, JP23.3, JP23.4, JP23.5, JP23.6, JP23.7, JP23.8
- new net N$6: J11.1, J11.2, J11.3, J11.4, J11.5, J11.6, J11.7, J11.8, J11.9
- new net N$7: J12.1, J12.2, J12.3, J12.4, J12.5, J12.6, J12.7, J12.8, J12.9
- new net N$8: J13.1, J13.2, J13.3, J13.4, J13.5, J13.6, J13.7, J13.8, J13.9
- new net N$9: J14.1, J14.2, J14.3, J14.4, J14.5, J14.6, J14.7, J14.8, J14.9
