File: xns-ip67-ESP12.brd (EAGLE design)
At the start: 65.3 x 129.3 mm, 195 parts, among them J1 DCJ0202

Commit message: Change FTDI Header
Change FTDI Header
Parts:
- removed PROG: (no value), con-lstb:MA03-1
- added JP37: (no value), pinhead:1X05
Connections:
- removed net N$20: MDL1.16, PROG.3
- new net N$13: JP37.4, MDL1.15
- new net N$7: JP23.1, JP23.2, JP23.3, JP23.4, JP23.5, JP23.6, JP23.7, JP23.8
- net GND: now also JP37.1; no longer PROG.1
- net N$4: now also JP37.5, MDL1.16; no longer MDL1.15, PROG.2
Routing:
- net N$4: track 27.6 -> 6.71 mm
- net N$7: track 0.00 -> 17.8 mm
- net N$20: track 16.4 -> 0.00 mm
- net N$13: track 0.00 -> 10.4 mm
Changed lines of the file:
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@@
 <wire x1="44.45" y1="60.96" x2="64.77" y2="60.96" width="0.4064" layer="25"/>
 <wire x1="64.77" y1="60.96" x2="64.77" y2="63.5" width="0.4064" layer="25"/>
-<text x="41.91" y="13.335" size="1.016" layer="27">RX</text>
-<text x="44.45" y="13.335" size="1.016" layer="27">GND</text>
-<text x="39.37" y="13.335" size="1.016" layer="27">TX</text>
+<text x="26.035" y="20.955" size="1.016" layer="27">RX</text>
+<text x="17.78" y="20.955" size="1.016" layer="27">GND</text>
+<text x="28.575" y="20.955" size="1.016" layer="27">TX</text>
 <text x="35.56" y="123.19" size="1.778" layer="25">xnsense.no</text>
 <text x="35.56" y="119.38" size="1.778" layer="25">xns-ip67-rev-0</text>
@@
 <attribute name="VALUE" x="63.5" y="23.46" size="0.0254" layer="27"/>
 </element>
-<element name="PROG" library="con-lstb" package="MA03-1" value="" x="43.18" y="11.43" smashed="yes" rot="R180">
-<attribute name="OC_NEWARK" value="unknown" x="43.18" y="11.43" size="1.778" layer="27" rot="R180" display="off"/>
-<attribute name="MF" value="" x="43.18" y="11.43" size="1.778" layer="27" rot="R180" display="off"/>
-<attribute name="MPN" value="" x="43.18" y="11.43" size="1.778" layer="27" rot="R180" display="off"/>
-<attribute name="OC_FARNELL" value="unknown" x="43.18" y="11.43" size="1.778" layer="27" rot="R180" display="off"/>
-<attribute name="VALUE" x="46.99" y="14.351" size="1.27" layer="27" ratio="10" rot="R180"/>
-</element>
 <element name="PAD71" library="wirepad" package="1,6/0,9" value="WIREPAD1,6/0,9" x="27.94" y="45.72" smashed="yes">
 <attribute name="VALUE" x="27.94" y="46.32" size="0.0254" layer="27"/>
@@
 <element name="PAD152" library="wirepad" package="1,6/0,9" value="WIREPAD1,6/0,9" x="17.78" y="27.94" smashed="yes">
 <attribute name="VALUE" x="17.78" y="28.54" size="0.0254" layer="27"/>
+</element>
+<element name="JP37" library="pinhead" package="1X05" value="" x="24.13" y="24.13" smashed="yes">
+<attribute name="VALUE" x="17.78" y="20.955" size="1.27" layer="27"/>
 </element>
 </elements>
@@
 <contactref element="JP32" pad="2"/>
 <contactref element="JP32" pad="1"/>
-<contactref element="PROG" pad="1"/>
 <polygon width="0.4064" layer="16">
 <vertex x="5.08" y="-2.54"/>
@@
 <wire x1="44.48" y1="4.585" x2="46.355" y2="4.585" width="0.508" layer="1"/>
 <wire x1="46.355" y1="4.585" x2="46.48" y2="4.71" width="0.508" layer="1"/>
+<contactref element="JP37" pad="1"/>
 </signal>
 <signal name="VCC">
@@
 <wire x1="55.626" y1="62.484" x2="55.88" y2="62.23" width="0.508" layer="1"/>
 </signal>
-<signal name="N$4">
-<contactref element="MDL1" pad="15"/>
-<contactref element="PROG" pad="2"/>
-<wire x1="34.29" y1="25.146" x2="35.052" y2="25.146" width="0.508" layer="1"/>
-<wire x1="33.528" y1="24.384" x2="34.29" y2="25.146" width="0.508" layer="1"/>
-<wire x1="33.528" y1="14.859" x2="33.528" y2="24.384" width="0.508" layer="1"/>
-<wire x1="40.767" y1="7.62" x2="33.528" y2="14.859" width="0.508" layer="1"/>
-<wire x1="42.291" y1="7.62" x2="40.767" y2="7.62" width="0.508" layer="1"/>
-<wire x1="43.053" y1="8.382" x2="42.291" y2="7.62" width="0.508" layer="1"/>
-<wire x1="43.053" y1="11.43" x2="43.053" y2="8.382" width="0.508" layer="1"/>
-<wire x1="35.052" y1="25.146" x2="35.08" y2="25.37" width="0.508" layer="1"/>
-<wire x1="43.053" y1="11.43" x2="43.18" y2="11.43" width="0.508" layer="1"/>
-</signal>
-<signal name="N$20">
-<contactref element="PROG" pad="3"/>
-<contactref element="MDL1" pad="16"/>
-<wire x1="34.29" y1="22.479" x2="35.052" y2="23.241" width="0.508" layer="1"/>
-<wire x1="34.29" y1="15.24" x2="34.29" y2="22.479" width="0.508" layer="1"/>
-<wire x1="38.1" y1="11.43" x2="34.29" y2="15.24" width="0.508" layer="1"/>
-<wire x1="40.64" y1="11.43" x2="38.1" y2="11.43" width="0.508" layer="1"/>
-<wire x1="35.052" y1="23.241" x2="35.08" y2="23.37" width="0.508" layer="1"/>
-</signal>
 <signal name="N$52">
 <via x="55.88" y="53.34" extent="1-16" drill="0.6"/>
@@
 </signal>
 <signal name="N$57">
-<via x="20.32" y="21.59" extent="1-16" drill="0.6"/>
+<via x="25.4" y="19.05" extent="1-16" drill="0.6"/>
 </signal>
 <signal name="N$58">
@@
 <wire x1="30.48" y1="43.434" x2="30.48" y2="43.18" width="0.508" layer="1"/>
 </signal>
+<signal name="N$7">
+<contactref element="JP23" pad="1"/>
+<contactref element="JP23" pad="2"/>
+<contactref element="JP23" pad="3"/>
+<contactref element="JP23" pad="4"/>
+<contactref element="JP23" pad="5"/>
+<contactref element="JP23" pad="6"/>
+<contactref element="JP23" pad="7"/>
+<contactref element="JP23" pad="8"/>
+<wire x1="45.72" y1="82.55" x2="48.26" y2="82.55" width="0.508" layer="1"/>
+<wire x1="48.26" y1="82.55" x2="50.8" y2="82.55" width="0.508" layer="1"/>
+<wire x1="50.8" y1="82.55" x2="53.34" y2="82.55" width="0.508" layer="1"/>
+<wire x1="53.34" y1="82.55" x2="55.88" y2="82.55" width="0.508" layer="1"/>
+<wire x1="55.88" y1="82.55" x2="58.42" y2="82.55" width="0.508" layer="1"/>
+<wire x1="58.42" y1="82.55" x2="60.96" y2="82.55" width="0.508" layer="1"/>
+<wire x1="60.96" y1="82.55" x2="63.5" y2="82.55" width="0.508" layer="1"/>
+</signal>
+<signal name="N$4">
+<contactref element="MDL1" pad="16"/>
+<contactref element="JP37" pad="5"/>
+<wire x1="29.21" y1="24.13" x2="30.48" y2="22.86" width="0.508" layer="1"/>
+<wire x1="30.48" y1="22.86" x2="32.385" y2="22.86" width="0.508" layer="1"/>
+<wire x1="32.385" y1="22.86" x2="33.02" y2="23.495" width="0.508" layer="1"/>
+<wire x1="33.02" y1="23.495" x2="34.955" y2="23.495" width="0.508" layer="1"/>
+<wire x1="34.955" y1="23.495" x2="35.08" y2="23.37" width="0.508" layer="1"/>
+</signal>
+<signal name="N$13">
+<contactref element="MDL1" pad="15"/>
+<contactref element="JP37" pad="4"/>
+<wire x1="26.67" y1="24.13" x2="26.67" y2="24.765" width="0.508" layer="1"/>
+<wire x1="26.67" y1="24.765" x2="28.575" y2="26.67" width="0.508" layer="1"/>
+<wire x1="28.575" y1="26.67" x2="32.385" y2="26.67" width="0.508" layer="1"/>
+<wire x1="32.385" y1="26.67" x2="33.655" y2="25.4" width="0.508" layer="1"/>
+<wire x1="33.655" y1="25.4" x2="35.05" y2="25.4" width="0.508" layer="1"/>
+<wire x1="35.05" y1="25.4" x2="35.08" y2="25.37" width="0.508" layer="1"/>
+</signal>
 </signals>
