File: xns-ip67-ESP12.brd (EAGLE design)
At the start: 65.3 x 129.3 mm, 195 parts, among them J1 DCJ0202

Commit message: Routed and Gerb files
Routed and produced verb files
Parts:
- removed 5.5V, PAD1, PAD10, PAD100, PAD101, PAD102, PAD103, PAD104, PAD105, PAD106, PAD107, PAD108, PAD109, PAD11, PAD110, PAD111, PAD112, PAD113, PAD114, PAD115, PAD116, PAD117, PAD118, PAD119, PAD12, PAD120, PAD121, PAD122, PAD123, PAD124, PAD125, PAD126, PAD127, PAD128, PAD129, PAD13, PAD130, PAD131, PAD132, PAD133, PAD134, PAD135, PAD136, PAD137, PAD138, PAD139, PAD14, PAD140, PAD141, PAD142, PAD143, PAD144, PAD145, PAD146, PAD147, PAD148, PAD149, PAD15, PAD150, PAD151, PAD152, PAD16, PAD17, PAD18, PAD19, PAD2, PAD20, PAD21, PAD22, PAD23, PAD24, PAD25, PAD26, PAD27, PAD28, PAD29, PAD3, PAD30, PAD31, PAD32, PAD33, PAD34, PAD35, PAD36, PAD37, PAD38, PAD39, PAD4, PAD40, PAD41, PAD42, PAD43, PAD44, PAD45, PAD46, PAD47, PAD48, PAD49, PAD5, PAD50, PAD51, PAD52, PAD53, PAD54, PAD55, PAD56, PAD57, PAD58, PAD59, PAD6, PAD60, PAD61, PAD62, PAD63, PAD64, PAD65, PAD66, PAD67, PAD68, PAD69, PAD7, PAD70, PAD71, PAD72, PAD73, PAD74, PAD75, PAD76, PAD77, PAD78, PAD79, PAD8, PAD80, PAD81, PAD82, PAD83, PAD84, PAD85, PAD86, PAD87, PAD88, PAD89, PAD9, PAD90, PAD91, PAD92, PAD93, PAD94, PAD95, PAD96, PAD97, PAD98, PAD99: WIREPAD1,6/0,9, wirepad:1,6/0,9
- removed MDL1: (no value), ESP8266-ESP12E:ESP8266-ESP12E
- added J10, J11, J12, J13, J18, J19, J2, J20, J21, J22, J23, J3, J4, J5, J6, J7, J8, J9: (no value), SparkFun-Connectors:1X06_NO_SILK
- added J14, J15, J16, J17: (no value), SparkFun-Connectors:1X11_NO_SILK
- added J24: 5V, SparkFun-Connectors:1X01_NO_SILK
- added J25, J26, J27, J28, J29, J30, J31, J32, J33, J34: (no value), SparkFun-Connectors:1X07_NO_SILK
- added X1: ESP-12E, microbuilder:ESP-12E
- moved U1 2.54 mm to (58.4, 6.35)
- moved X2 0.99 mm to (43.2, 2.82)
Connections:
- new net N$20: J22.1, J22.2, J22.3, J22.4, J22.5, J22.6
- new net N$52: J31.1, J31.2, J31.3, J31.4, J31.5, J31.6, J31.7
- new net N$54: J32.1, J32.2, J32.3, J32.4, J32.5, J32.6, J32.7
- new net N$56: J33.1, J33.2, J33.3, J33.4, J33.5, J33.6, J33.7
- new net N$58: J34.1, J34.2, J34.3, J34.4, J34.5, J34.6, J34.7
- new net N$71: J25.1, J25.2, J25.3, J25.4, J25.5, J25.6, J25.7
- new net N$73: J27.1, J27.2, J27.3, J27.4, J27.5, J27.6, J27.7
- new net N$74: J28.1, J28.2, J28.3, J28.4, J28.5, J28.6, J28.7
- new net N$75: J29.1, J29.2, J29.3, J29.4, J29.5, J29.6, J29.7
- new net N$76: J30.1, J30.2, J30.3, J30.4, J30.5, J30.6, J30.7
- net GND: now also J14.1, J14.10, J14.11, J14.2, J14.3, J14.4, J14.5, J14.6, J14.7, J14.8, J14.9, J16.1, J16.10, J16.11, J16.2, J16.3, J16.4, J16.5, J16.6, J16.7, J16.8, J16.9, X1.9; no longer MDL1.9, PAD1.1, PAD107.1, PAD108.1, PAD109.1, PAD110.1, PAD111.1, PAD13.1, PAD14.1, PAD15.1, PAD16.1, PAD17.1, PAD18.1, PAD19.1, PAD2.1, PAD25.1, PAD26.1, PAD3.1, PAD39.1, PAD4.1, PAD40.1, PAD5.1, PAD6.1
- net N$1: now also J2.1, J2.2, J2.3, J2.4, J2.5, J2.6, X1.7; no longer MDL1.19, PAD117.1, PAD118.1, PAD27.1, PAD28.1, PAD29.1, PAD30.1
- net N$10: now also J9.1, J9.2, J9.3, J9.4, J9.5, J9.6, X1.10; no longer MDL1.2, PAD133.1, PAD136.1, PAD63.1, PAD64.1, PAD65.1, PAD66.1
- net N$11: now also J10.1, J10.2, J10.3, J10.4, J10.5, J10.6, X1.11; no longer MDL1.1, PAD134.1, PAD135.1, PAD67.1, PAD68.1, PAD69.1, PAD70.1
- net N$12: now also J11.1, J11.2, J11.3, J11.4, J11.5, J11.6, X1.12; no longer MDL1.20, PAD137.1, PAD138.1, PAD71.1, PAD72.1, PAD73.1, PAD74.1
- net N$13: now also X1.15; no longer MDL1.15
- net N$14: now also J12.1, J12.2, J12.3, J12.4, J12.5, J12.6, X1.13; no longer MDL1.22, PAD141.1, PAD142.1, PAD79.1, PAD80.1, PAD81.1, PAD82.1
- net N$15: now also J13.1, J13.2, J13.3, J13.4, J13.5, J13.6, X1.14; no longer MDL1.10, PAD143.1, PAD144.1, PAD83.1, PAD84.1, PAD85.1, PAD86.1
- net N$16: now also J18.1, J18.2, J18.3, J18.4, J18.5, J18.6; no longer MDL1.11, PAD145.1, PAD146.1, PAD87.1, PAD88.1, PAD89.1, PAD90.1
- net N$17: now also J19.1, J19.2, J19.3, J19.4, J19.5, J19.6; no longer MDL1.12, PAD147.1, PAD148.1, PAD91.1, PAD92.1, PAD93.1, PAD94.1
- net N$18: now also J20.1, J20.2, J20.3, J20.4, J20.5, J20.6; no longer MDL1.13, PAD149.1, PAD150.1, PAD95.1, PAD96.1, PAD97.1, PAD98.1
- net N$19: now also J21.1, J21.2, J21.3, J21.4, J21.5, J21.6; no longer MDL1.14, PAD100.1, PAD101.1, PAD102.1, PAD151.1, PAD152.1, PAD99.1
- net N$2: now also J3.1, J3.2, J3.3, J3.4, J3.5, J3.6, X1.6; no longer MDL1.18, PAD119.1, PAD120.1, PAD31.1, PAD32.1, PAD33.1, PAD34.1
- net N$3: now also J4.1, J4.2, J4.3, J4.4, J4.5, J4.6, X1.5; no longer MDL1.17, PAD121.1, PAD122.1, PAD35.1, PAD36.1, PAD37.1, PAD38.1
- net N$4: now also X1.16; no longer MDL1.16
- net N$5: now also J5.1, J5.2, J5.3, J5.4, J5.5, J5.6, X1.4; no longer MDL1.7, PAD123.1, PAD124.1, PAD43.1, PAD44.1, PAD45.1, PAD46.1
- net N$6: now also J6.1, J6.2, J6.3, J6.4, J6.5, J6.6, X1.3; no longer MDL1.6, PAD125.1, PAD126.1, PAD47.1, PAD48.1, PAD49.1, PAD50.1
- net N$70: now also J23.1, J23.2, J23.3, J23.4, J23.5, J23.6; no longer MDL1.21, PAD139.1, PAD140.1, PAD75.1, PAD76.1, PAD77.1, PAD78.1
- net N$72: now also J26.1, J26.2, J26.3, J26.4, J26.5, J26.6, J26.7; no longer MDL1.5, PAD127.1, PAD128.1, PAD51.1, PAD52.1, PAD53.1, PAD54.1
- net N$8: now also J7.1, J7.2, J7.3, J7.4, J7.5, J7.6, X1.2; no longer MDL1.4, PAD129.1, PAD130.1, PAD55.1, PAD56.1, PAD57.1, PAD58.1
- net N$9: now also J8.1, J8.2, J8.3, J8.4, J8.5, J8.6, X1.1; no longer MDL1.3, PAD131.1, PAD132.1, PAD59.1, PAD60.1, PAD61.1, PAD62.1
- net VCC: now also J24.1; no longer 5.5V.1
- net VDD: now also J15.1, J15.10, J15.11, J15.2, J15.3, J15.4, J15.5, J15.6, J15.7, J15.8, J15.9, J17.1, J17.10, J17.11, J17.2, J17.3, J17.4, J17.5, J17.6, J17.7, J17.8, J17.9, X1.8; no longer MDL1.8, PAD10.1, PAD103.1, PAD104.1, PAD105.1, PAD106.1, PAD11.1, PAD112.1, PAD113.1, PAD114.1, PAD115.1, PAD116.1, PAD12.1, PAD20.1, PAD21.1, PAD22.1, PAD23.1, PAD24.1, PAD41.1, PAD42.1, PAD7.1, PAD8.1, PAD9.1
Routing:
- net GND: track 49.4 -> 7.64 mm, vias 4 -> 17
- net N$54: track 0.00 -> 17.1 mm, vias 1 -> 0
- net N$73: track 0.00 -> 16.8 mm
- net N$76: track 0.00 -> 16.0 mm
- net N$56: track 0.00 -> 16.0 mm, vias 1 -> 0
- net N$74: track 0.00 -> 15.8 mm
- net N$71: track 0.00 -> 15.8 mm
- net N$75: track 0.00 -> 15.2 mm
- net N$58: track 0.00 -> 15.2 mm, vias 1 -> 0
- net N$52: track 0.00 -> 15.2 mm, vias 1 -> 0
- net N$20: track 0.00 -> 14.2 mm
- net N$70: track 25.8 -> 13.3 mm
- net VCC: track 55.8 -> 46.3 mm, vias 0 -> 1
- net N$1: track 27.1 -> 19.0 mm
- net N$12: track 26.8 -> 19.1 mm
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Other:
- board text added: "ADC"
- board text added: "CHPD"
- board text added: "D0"
- board text added: "D12"
- board text added: "D13"
- board text added: "D14"
- board text added: "D15"
- board text added: "D16"
- board text added: "D2"
- board text added: "D4"
- board text added: "D5"
- board text added: "RST"
- board text added: "xns ip67-ESP12 rev 1"
- board text removed: "xns-ip67-ESP12-rev-0"
