File: xns-ip67-ESP12-New.brd (EAGLE design)
At the start: 65.3 x 130.5 mm, 67 parts, among them J1 DCJ0202

Commit message: New board layout
New board layout
Parts:
- removed 5.5V: WIREPAD1,6/0,9, wirepad:1,6/0,9
- added J28, J29, J30, J31, J32, J33, J34: (no value), SparkFun-Connectors:1X07_NO_SILK
- added JP37: (no value), pinhead:1X05
- added X1: ESP-12E, microbuilder:ESP-12E
- J10, J11, J12, J13, J18, J19, J20, J21, J22, J23, J6, J7, J8, J9: device SparkFun-Connectors:1X09_NO_SILK -> SparkFun-Connectors:1X06_NO_SILK
- J14, J15, J16, J17: device SparkFun-Connectors:1X09_NO_SILK -> SparkFun-Connectors:1X11_NO_SILK
- J2, J3, J4, J5: device SparkFun-Connectors:1X11_NO_SILK -> SparkFun-Connectors:1X06_NO_SILK
- J24: value (none) -> 5V; device SparkFun-Connectors:1X09_NO_SILK -> SparkFun-Connectors:1X01_NO_SILK
- J25, J26, J27: device SparkFun-Connectors:1X09_NO_SILK -> SparkFun-Connectors:1X07_NO_SILK
- moved J17 57.4 mm to (71.1, 20.3), turned to 90 degrees
- moved J2 45.0 mm to (55.9, 38.1), turned to 0 degrees
- moved J3 41.8 mm to (55.9, 35.6), turned to 0 degrees
- moved J21 36.7 mm to (55.9, 45.7)
- moved J22 36.7 mm to (55.9, 43.2)
- moved J23 36.7 mm to (55.9, 40.6)
- moved J14 33.6 mm to (12.7, 20.3), turned to 90 degrees
- moved J25 33.4 mm to (25.4, 59.7)
- moved J26 33.4 mm to (25.4, 57.1)
- moved J27 33.4 mm to (25.4, 54.6)
- moved J15 30.7 mm to (15.2, 20.3), turned to 90 degrees
- moved J10 28.0 mm to (17.8, 35.6)
- moved J11 28.0 mm to (17.8, 33.0)
- moved J12 28.0 mm to (17.8, 30.5)
- moved J13 28.0 mm to (17.8, 27.9)
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Connections:
- removed net N$53: J27.1, J27.2, J27.3, J27.4, J27.5, J27.6, J27.7, J27.8, J27.9
- removed net N$7 (its old number): J12.1, J12.2, J12.3, J12.4, J12.5, J12.6, J12.7, J12.8, J12.9
- new net N$54: J32.1, J32.2, J32.3, J32.4, J32.5, J32.6, J32.7
- new net N$56: J33.1, J33.2, J33.3, J33.4, J33.5, J33.6, J33.7
- new net N$58: J34.1, J34.2, J34.3, J34.4, J34.5, J34.6, J34.7
- new net N$70: J23.1, J23.2, J23.3, J23.4, J23.5, J23.6
- new net N$71: J25.1, J25.2, J25.3, J25.4, J25.5, J25.6, J25.7
- new net N$72: J26.1, J26.2, J26.3, J26.4, J26.5, J26.6, J26.7
- new net N$73: J27.1, J27.2, J27.3, J27.4, J27.5, J27.6, J27.7
- new net N$74: J28.1, J28.2, J28.3, J28.4, J28.5, J28.6, J28.7
- new net N$75: J29.1, J29.2, J29.3, J29.4, J29.5, J29.6, J29.7
- new net N$76: J30.1, J30.2, J30.3, J30.4, J30.5, J30.6, J30.7
- net GND: now also J14.1, J14.10, J14.11, J14.2, J14.3, J14.4, J14.5, J14.6, J14.7, J14.8, J14.9, J16.1, J16.10, J16.11, J16.2, J16.3, J16.4, J16.5, J16.6, J16.7, J16.8, J16.9, JP37.1, X1.9; no longer J2.1, J2.10, J2.11, J2.2, J2.3, J2.4, J2.5, J2.6, J2.7, J2.8, J2.9, J4.1, J4.10, J4.11, J4.2, J4.3, J4.4, J4.5, J4.6, J4.7, J4.8, J4.9
- net N$1: now also J2.1, J2.2, J2.3, J2.4, J2.5, J2.6, X1.7; no longer J6.1, J6.2, J6.3, J6.4, J6.5, J6.6, J6.7, J6.8, J6.9
- net N$10: now also J9.1, J9.2, J9.3, J9.4, J9.5, J9.6, X1.10; no longer J15.1, J15.2, J15.3, J15.4, J15.5, J15.6, J15.7, J15.8, J15.9
- net N$11: now also J10.1, J10.2, J10.3, J10.4, J10.5, J10.6, X1.11; no longer J16.1, J16.2, J16.3, J16.4, J16.5, J16.6, J16.7, J16.8, J16.9
- net N$12: now also J11.1, J11.2, J11.3, J11.4, J11.5, J11.6, X1.12; no longer J17.1, J17.2, J17.3, J17.4, J17.5, J17.6, J17.7, J17.8, J17.9
- net N$13: now also JP37.4, X1.15; no longer J18.1, J18.2, J18.3, J18.4, J18.5, J18.6, J18.7, J18.8, J18.9
- net N$14: now also J12.1, J12.2, J12.3, J12.4, J12.5, J12.6, X1.13; no longer J19.1, J19.2, J19.3, J19.4, J19.5, J19.6, J19.7, J19.8, J19.9
- net N$15: now also J13.1, J13.2, J13.3, J13.4, J13.5, J13.6, X1.14; no longer J20.1, J20.2, J20.3, J20.4, J20.5, J20.6, J20.7, J20.8, J20.9
- net N$16: now also J18.1, J18.2, J18.3, J18.4, J18.5, J18.6; no longer J21.1, J21.2, J21.3, J21.4, J21.5, J21.6, J21.7, J21.8, J21.9
- net N$17: now also J19.1, J19.2, J19.3, J19.4, J19.5, J19.6; no longer J22.1, J22.2, J22.3, J22.4, J22.5, J22.6, J22.7, J22.8, J22.9
- net N$18: now also J20.1, J20.2, J20.3, J20.4, J20.5, J20.6; no longer J23.1, J23.2, J23.3, J23.4, J23.5, J23.6, J23.7, J23.8, J23.9
- net N$19: now also J21.1, J21.2, J21.3, J21.4, J21.5, J21.6; no longer J24.1, J24.2, J24.3, J24.4, J24.5, J24.6, J24.7, J24.8, J24.9
- net N$2: now also J3.1, J3.2, J3.3, J3.4, J3.5, J3.6, X1.6; no longer J7.1, J7.2, J7.3, J7.4, J7.5, J7.6, J7.7, J7.8, J7.9
- net N$20: now also J22.1, J22.2, J22.3, J22.4, J22.5, J22.6; no longer J25.1, J25.2, J25.3, J25.4, J25.5, J25.6, J25.7, J25.8, J25.9
- net N$3: now also J4.1, J4.2, J4.3, J4.4, J4.5, J4.6, X1.5; no longer J8.1, J8.2, J8.3, J8.4, J8.5, J8.6, J8.7, J8.8, J8.9
- net N$4: now also JP37.5, X1.16; no longer J9.1, J9.2, J9.3, J9.4, J9.5, J9.6, J9.7, J9.8, J9.9
- net N$5: now also J5.1, J5.2, J5.3, J5.4, J5.5, J5.6, X1.4; no longer J10.1, J10.2, J10.3, J10.4, J10.5, J10.6, J10.7, J10.8, J10.9
- net N$52: now also J31.1, J31.2, J31.3, J31.4, J31.5, J31.6, J31.7; no longer J26.1, J26.2, J26.3, J26.4, J26.5, J26.6, J26.7, J26.8, J26.9
- net N$6: now also J6.1, J6.2, J6.3, J6.4, J6.5, J6.6, X1.3; no longer J11.1, J11.2, J11.3, J11.4, J11.5, J11.6, J11.7, J11.8, J11.9
- net N$8: now also J7.1, J7.2, J7.3, J7.4, J7.5, J7.6, X1.2; no longer J13.1, J13.2, J13.3, J13.4, J13.5, J13.6, J13.7, J13.8, J13.9
- net N$9: now also J8.1, J8.2, J8.3, J8.4, J8.5, J8.6, X1.1; no longer J14.1, J14.2, J14.3, J14.4, J14.5, J14.6, J14.7, J14.8, J14.9
- net VCC: now also J24.1; no longer 5.5V.1
- net VDD: now also J15.1, J15.10, J15.11, J15.2, J15.3, J15.4, J15.5, J15.6, J15.7, J15.8, J15.9, J17.1, J17.10, J17.11, J17.2, J17.3, J17.4, J17.5, J17.6, J17.7, J17.8, J17.9, X1.8; no longer J3.1, J3.10, J3.11, J3.2, J3.3, J3.4, J3.5, J3.6, J3.7, J3.8, J3.9, J5.1, J5.10, J5.11, J5.2, J5.3, J5.4, J5.5, J5.6, J5.7, J5.8, J5.9
Routing:
- net VCC: track 77.4 -> 46.3 mm
- net N$7 (its old number): track 22.5 -> 0.00 mm
- net VDD: track 287.6 -> 265.9 mm
- net N$53: track 21.1 -> 0.00 mm
- net N$54: track 0.00 -> 17.1 mm
- net N$73: track 0.00 -> 16.8 mm
- net N$76: track 0.00 -> 16.0 mm
- net N$56: track 0.00 -> 16.0 mm
- net N$74: track 0.00 -> 15.8 mm
- net N$71: track 0.00 -> 15.8 mm
- net N$4: track 22.5 -> 6.76 mm
- net N$75: track 0.00 -> 15.2 mm
- net N$72: track 0.00 -> 15.2 mm
- net N$58: track 0.00 -> 15.2 mm
- net N$70: track 0.00 -> 13.3 mm
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Other:
- board size 65.3 x 130.5 mm -> 65.3 x 132.3 mm
- board text added: "ADC"
- board text added: "CHPD"
- board text added: "D0"
- board text added: "D12"
- board text added: "D13"
- board text added: "D14"
- board text added: "D15"
- board text added: "D16"
- board text added: "D2"
- board text added: "D4"
- board text added: "D5"
- board text added: "RST"
- board text added: "RX"
- board text added: "TX"
- board text added: "xns ip67-ESP12 rev 1"
- board text removed: "xns ip67 rev 1"
