File: xns-ip67.brd (EAGLE design)
At the start: 65.3 x 129.3 mm, 67 parts, among them J1 DCJ0202

Commit message: Change square via to round
Change square via to round
Routing:
- net VDD: track 287.6 -> 281.9 mm
Other:
- board size 65.3 x 129.3 mm -> 65.3 x 130.5 mm
Changed lines of the file:
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@@
 <?xml version="1.0" encoding="utf-8"?>
 <!DOCTYPE eagle SYSTEM "eagle.dtd">
-<eagle version="7.7.0">
+<eagle version="8.0.0">
 <drawing>
 <settings>
@@
 <setting verticaltext="up"/>
 </settings>
-<grid distance="1.27" unitdist="mm" unit="mil" style="lines" multiple="1" display="yes" altdistance="12.5" altunitdist="mil" altunit="mil"/>
+<grid distance="5" unitdist="mil" unit="mil" style="lines" multiple="1" display="yes" altdistance="1" altunitdist="mil" altunit="mil"/>
 <layers>
 <layer number="1" name="Top" color="4" fill="1" visible="yes" active="yes"/>
@@
 <wire x1="25.4428" y1="127.7886" x2="60.8504" y2="127.7886" width="0.1" layer="20"/>
 <wire x1="61.9172" y1="127.306" x2="60.8504" y2="127.783646875" width="0.1" layer="20" curve="48.2397"/>
-<wire x1="60.8504" y1="-1.472" x2="61.905159375" y2="-1.00390625" width="0.0254" layer="20" curve="47.862401"/>
-<wire x1="60.8504" y1="-1.472" x2="25.4428" y2="-1.472" width="0.0254" layer="20"/>
-<wire x1="24.376" y1="-1.0148" x2="25.4428" y2="-1.492446875" width="0.0254" layer="20" curve="48.2397"/>
 <wire x1="64.22" y1="120.7" x2="64.22" y2="125.56" width="0.1" layer="20"/>
 <wire x1="60.84" y1="127.79" x2="60.86" y2="127.79" width="0.1" layer="20"/>
@@
 <wire x1="64.12" y1="0.7" x2="64.03" y2="0.65" width="0.1" layer="20"/>
 <wire x1="64.03" y1="0.65" x2="62.01" y2="-0.9" width="0.1" layer="20" curve="16.890774"/>
-<wire x1="62.01" y1="-0.9" x2="61.64" y2="-1.23" width="0.1" layer="20" curve="-8.431762"/>
-<wire x1="61.64" y1="-1.23" x2="61.37" y2="-1.38" width="0.1" layer="20" curve="-16.91809"/>
-<wire x1="61.37" y1="-1.38" x2="60.92" y2="-1.47" width="0.1" layer="20" curve="-18.571066"/>
-<wire x1="60.92" y1="-1.47" x2="25.45" y2="-1.47" width="0.1" layer="20"/>
-<wire x1="25.45" y1="-1.47" x2="24.23" y2="-0.87" width="0.1" layer="20" curve="-52.376191"/>
+<wire x1="60.92" y1="-2.74" x2="25.4754" y2="-2.74" width="0.1" layer="20"/>
 <wire x1="24.23" y1="-0.87" x2="23.89" y2="-0.51" width="0.1" layer="20" curve="11.479415"/>
 <wire x1="23.89" y1="-0.51" x2="22.18" y2="0.68" width="0.1" layer="20" curve="9.974227"/>
@@
 <wire x1="41.91" y1="25.4" x2="41.91" y2="22.86" width="0.4064" layer="25"/>
 <wire x1="41.91" y1="22.86" x2="19.05" y2="22.86" width="0.4064" layer="25"/>
+<wire x1="24.1935" y1="-0.8255" x2="25.4635" y2="-2.7305" width="0.1" layer="20"/>
+<wire x1="62.0141" y1="-0.889" x2="60.9346" y2="-2.7432" width="0.1" layer="20"/>
 </plain>
 <attributes>
@@
 <wire x1="29.718" y1="11.938" x2="33.02" y2="15.24" width="0.508" layer="16"/>
 <wire x1="33.02" y1="15.24" x2="38.1" y2="15.24" width="0.508" layer="16"/>
-<via x="38.1" y="15.24" extent="1-16" drill="0.508" shape="square"/>
+<via x="38.1" y="15.24" extent="1-16" drill="0.508"/>
 <wire x1="38.1" y1="15.24" x2="38.1" y2="10.16" width="0.508" layer="1"/>
 <wire x1="38.1" y1="10.16" x2="41.91" y2="6.35" width="0.508" layer="1"/>
@@
 <wire x1="20.32" y1="17.78" x2="43.18" y2="17.78" width="0.508" layer="16"/>
 <wire x1="43.18" y1="17.78" x2="46.99" y2="13.97" width="0.508" layer="16"/>
-<via x="46.99" y="13.97" extent="1-16" drill="0.508" shape="square"/>
+<via x="46.99" y="13.97" extent="1-16" drill="0.508"/>
 <wire x1="46.99" y1="13.97" x2="47.44" y2="13.97" width="0.508" layer="1"/>
 <wire x1="47.44" y1="13.97" x2="53.81" y2="7.6" width="0.508" layer="1"/>
 <wire x1="67.945" y1="72.39" x2="67.945" y2="67.945" width="0.508" layer="16"/>
-<wire x1="67.945" y1="67.945" x2="66.04" y2="66.04" width="0.508" layer="16"/>
-<wire x1="66.04" y1="66.04" x2="66.04" y2="63.5" width="0.508" layer="16"/>
-<via x="66.04" y="63.5" extent="1-16" drill="0.508" shape="square"/>
-<wire x1="66.04" y1="63.5" x2="44.1325" y2="63.5" width="0.508" layer="1"/>
-<wire x1="44.1325" y1="63.5" x2="43.65625" y2="63.02375" width="0.508" layer="1"/>
-<wire x1="43.65625" y1="63.02375" x2="43.4975" y2="62.865" width="0.508" layer="1"/>
-<wire x1="43.4975" y1="62.865" x2="43.4975" y2="46.6725" width="0.508" layer="1"/>
-<wire x1="43.4975" y1="46.6725" x2="44.45" y2="45.72" width="0.508" layer="1"/>
-<wire x1="44.45" y1="45.72" x2="68.58" y2="45.72" width="0.508" layer="1"/>
-<wire x1="68.58" y1="45.72" x2="69.85" y2="46.99" width="0.508" layer="1"/>
+<wire x1="67.945" y1="67.945" x2="67.691" y2="66.167" width="0.508" layer="16"/>
+<wire x1="67.691" y1="66.167" x2="66.04" y2="63.5" width="0.508" layer="16"/>
+<via x="66.04" y="63.5" extent="1-16" drill="0.508"/>
+<wire x1="66.04" y1="63.5" x2="44.6405" y2="63.5" width="0.508" layer="1"/>
+<wire x1="44.6405" y1="63.5" x2="43.22445" y2="62.36335" width="0.508" layer="1"/>
+<wire x1="43.22445" y1="62.36335" x2="43.2435" y2="60.96" width="0.508" layer="1"/>
+<wire x1="43.2435" y1="60.96" x2="43.2435" y2="51.7525" width="0.508" layer="1"/>
+<wire x1="43.2435" y1="51.7525" x2="48.006" y2="49.149" width="0.508" layer="1"/>
+<wire x1="48.006" y1="49.149" x2="67.691" y2="49.149" width="0.508" layer="1"/>
+<wire x1="67.691" y1="49.149" x2="69.85" y2="46.99" width="0.508" layer="1"/>
 <wire x1="18.415" y1="72.39" x2="18.415" y2="69.215" width="0.508" layer="1"/>
-<wire x1="18.415" y1="69.215" x2="20.32" y2="67.31" width="0.508" layer="1"/>
-<wire x1="20.32" y1="67.31" x2="20.32" y2="63.5" width="0.508" layer="1"/>
-<wire x1="20.32" y1="63.5" x2="43.18" y2="63.5" width="0.508" layer="1"/>
-<wire x1="43.18" y1="63.5" x2="43.65625" y2="63.02375" width="0.508" layer="1"/>
+<wire x1="18.415" y1="69.215" x2="18.542" y2="66.929" width="0.508" layer="1"/>
+<wire x1="18.542" y1="66.929" x2="21.59" y2="63.5" width="0.508" layer="1"/>
+<wire x1="21.59" y1="63.5" x2="42.037" y2="63.5" width="0.508" layer="1"/>
+<wire x1="42.037" y1="63.5" x2="43.22445" y2="62.36335" width="0.508" layer="1"/>
 <wire x1="18.415" y1="90.17" x2="18.415" y2="92.71" width="0" layer="19" extent="1-1"/>
 </signal>
