File: xns-ip67-ESP12-New.sch (EAGLE design)
At the start: 75 parts, among them J1 DCJ0202, J24 5V, X1 ESP-12E

Commit message: Board dimension changes
Adjusted to be edge to edge
Parts:
- renumbered DC1 to DC3V3
Changed lines of the file:
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@@
 <?xml version="1.0" encoding="utf-8"?>
 <!DOCTYPE eagle SYSTEM "eagle.dtd">
-<eagle version="7.7.0">
+<eagle version="8.0.0">
 <drawing>
 <settings>
@@
 </classes>
 <parts>
-<part name="DC1" library="dc-dc-converter" deviceset="R-78C*-1.0" device="" technology="1.8"/>
+<part name="DC3V3" library="dc-dc-converter" deviceset="R-78C*-1.0" device="" technology="1.8"/>
 <part name="P+1" library="supply1" deviceset="VCC" device=""/>
 <part name="SUPPLY1" library="supply2" deviceset="VDD" device=""/>
@@
 </plain>
 <instances>
-<instance part="DC1" gate="G$1" x="68.58" y="121.92"/>
+<instance part="DC3V3" gate="G$1" x="68.58" y="121.92"/>
 <instance part="P+1" gate="VCC" x="50.8" y="127"/>
 <instance part="SUPPLY1" gate="G$1" x="86.36" y="124.46"/>
@@
 <net name="VCC" class="0">
 <segment>
-<pinref part="DC1" gate="G$1" pin="VIN"/>
+<pinref part="DC3V3" gate="G$1" pin="VIN"/>
 <wire x1="55.88" y1="121.92" x2="50.8" y2="121.92" width="0.1524" layer="91"/>
 <pinref part="P+1" gate="VCC" pin="VCC"/>
@@
 <net name="GND" class="0">
 <segment>
-<pinref part="DC1" gate="G$1" pin="GND"/>
+<pinref part="DC3V3" gate="G$1" pin="GND"/>
 <pinref part="GND1" gate="1" pin="GND"/>
 <wire x1="68.58" y1="114.3" x2="68.58" y2="111.76" width="0.1524" layer="91"/>
@@
 <pinref part="JP31" gate="G$1" pin="1"/>
 <wire x1="180.34" y1="162.56" x2="180.34" y2="165.1" width="0.1524" layer="91"/>
+<junction x="180.34" y="137.16"/>
+<junction x="180.34" y="139.7"/>
+<junction x="180.34" y="142.24"/>
+<junction x="180.34" y="144.78"/>
+<junction x="180.34" y="147.32"/>
+<junction x="180.34" y="149.86"/>
+<junction x="180.34" y="152.4"/>
+<junction x="180.34" y="154.94"/>
+<junction x="180.34" y="157.48"/>
+<junction x="180.34" y="160.02"/>
+<junction x="180.34" y="162.56"/>
+<junction x="180.34" y="165.1"/>
 </segment>
 <segment>
@@
 <pinref part="JP32" gate="G$1" pin="1"/>
 <wire x1="195.58" y1="162.56" x2="195.58" y2="165.1" width="0.1524" layer="91"/>
+<junction x="195.58" y="165.1"/>
+<junction x="195.58" y="162.56"/>
+<junction x="195.58" y="160.02"/>
+<junction x="195.58" y="157.48"/>
+<junction x="195.58" y="154.94"/>
+<junction x="195.58" y="152.4"/>
+<junction x="195.58" y="149.86"/>
+<junction x="195.58" y="147.32"/>
+<junction x="195.58" y="144.78"/>
+<junction x="195.58" y="142.24"/>
+<junction x="195.58" y="139.7"/>
+<junction x="195.58" y="137.16"/>
 </segment>
 <segment>
@@
 <net name="VDD" class="0">
 <segment>
-<pinref part="DC1" gate="G$1" pin="VOUT"/>
+<pinref part="DC3V3" gate="G$1" pin="VOUT"/>
 <pinref part="SUPPLY1" gate="G$1" pin="VDD"/>
 <wire x1="81.28" y1="121.92" x2="86.36" y2="121.92" width="0.1524" layer="91"/>
@@
 </sheet>
 </sheets>
-<errors>
-</errors>
 </schematic>
 </drawing>

Commit message: Added LiPo charging (new)
Components are not aligned etc, just added based on feather board. No
other components has been removed.
Parts:
- removed J24: 5V, SparkFun-Connectors:M01PTH_NO_SILK_YES_STOP
- removed X2: (no value), microbuilder:USBMICRO_20329
- added C3, C4: 10uF, capacitor-wima:C2.5/2
- added CN2: JSTPH, microbuilder:JST_2PIN
- added LED1: RED, microbuilder:LED0805_NOOUTLINE
- added LED2: GREEN, microbuilder:LED0805_NOOUTLINE
- added R5, R6: 470, eagle-ltspice:R0204/7
- added R7: 10k, eagle-ltspice:R0204/7
- added R8: 2.5k, eagle-ltspice:R0204/7
- added SJ1: (no value), microbuilder:SOLDERJUMPER
- added U2: MCP73831T-2ACI/OT, microbuilder:MCP73831/2
- added X3: (no value), jcbrataas:USB
- added X4: (no value), microbuilder:USB_MICRO_20329_V2
Connections:
- new net N$53: LED1.C, R5.1
- new net N$55: R5.2, R6.2, U2.STAT
- new net N$57: R7.1, SJ1.2, U2.PROG
- new net N$59: LED2.A, R6.1
- new net N$60: R8.1, SJ1.1
- new net VBAT1: C4.1, CN2.2, U2.VBAT
- new net VDD1: C3.1, LED1.A, U2.VDD, X4.VBUS
- net GND: now also C3.2, C4.2, CN2.1, LED2.C, R7.2, R8.2, U2.VSS, X3.GND, X4.GND; no longer X2.GND
- net VCC: now also X3.VBUS; no longer J24.1, X2.VBUS
Other:
- note added: "1.0K = 1000mA"
- note added: "10K = 100mA"
- note added: "2.0K = 500mA"
- note added: "5.0K = 200mA"
