File: xns-ip67-ESP12-New.sch (EAGLE design)
At the start: 86 parts, among them CN2 JSTPH, J1 DCJ0202, U2 MCP73831T-2ACI/OT, X1 ESP-12E

Commit message: ip67 version with A7, SIM, SMA
Test version with A7, SIM Card Holder and SMA Antenna
Parts:
- removed C3: 10uF, capacitor-wima:C2.5/2
- removed J11, J6, J8, J9: (no value), SparkFun-Connectors:M06NO_SILK_FEMALE_PTH
- removed JP16, JP17, JP18, JP19, JP20, JP21, JP22, JP23, JP24, JP5, JP6, JP7, JP8, JP9: (no value), adafruit:PINHD-1X8CLEANBIG
- removed LED1: RED, microbuilder:LED0805_NOOUTLINE
- removed LED2: GREEN, microbuilder:LED0805_NOOUTLINE
- removed R5: 470, eagle-ltspice:R0204/7
- removed R8: 2.5k, eagle-ltspice:R0204/7
- removed SJ1: (no value), microbuilder:SOLDERJUMPER
- removed U1: (no value), SparkFun-PowerIC:MIC52053.3V
- removed X4: (no value), microbuilder:USB_MICRO_20329_V2
- added D1: 1N4148, SparkFun-DiscreteSemi:DIODE1N4148
- added JCB_MICROUSB: (no value), jcbrataas-2:USB
- added LED4: Orange, adafruit:LED5MM
- added R1, R2, R3, R4: 10k, eagle-ltspice:R0204/7
- added R250: (no value), eagle-ltspice:R0204/7
- added SIMCARD: (no value), SparkFun-Connectors:SIMHOLDERSIM
- added STD_MICROUSB: (no value), microbuilder:USB_MICRO_20329_V2
- added U3: A7, IC:A7
- added X5: (no value), adafruit:SMACONNECTOR
- JP1, JP2, JP3, JP4: device adafruit:PINHD-1X8CLEANBIG -> adafruit:PINHD-1X1CB
- R6: value 470 -> 470k
- X3: device jcbrataas:USB -> adafruit:SMACONNECTOR_EDGE
Connections:
- net N$13 renamed RX
- net N$4 renamed TX
- removed net N$25: JP5.1, JP5.2, JP5.3, JP5.4, JP5.5, JP5.6, JP5.7, JP5.8
- removed net N$26: JP6.1, JP6.2, JP6.3, JP6.4, JP6.5, JP6.6, JP6.7, JP6.8
- removed net N$27: JP7.1, JP7.2, JP7.3, JP7.4, JP7.5, JP7.6, JP7.7, JP7.8
- removed net N$28: JP8.1, JP8.2, JP8.3, JP8.4, JP8.5, JP8.6, JP8.7, JP8.8
- removed net N$29: JP9.1, JP9.2, JP9.3, JP9.4, JP9.5, JP9.6, JP9.7, JP9.8
- removed net N$42: JP24.1, JP24.2, JP24.3, JP24.4, JP24.5, JP24.6, JP24.7, JP24.8
- removed net N$43: JP22.1, JP22.2, JP22.3, JP22.4, JP22.5, JP22.6, JP22.7, JP22.8
- removed net N$44: JP21.1, JP21.2, JP21.3, JP21.4, JP21.5, JP21.6, JP21.7, JP21.8
- removed net N$45: JP20.1, JP20.2, JP20.3, JP20.4, JP20.5, JP20.6, JP20.7, JP20.8
- removed net N$46: JP19.1, JP19.2, JP19.3, JP19.4, JP19.5, JP19.6, JP19.7, JP19.8
- removed net N$47: JP18.1, JP18.2, JP18.3, JP18.4, JP18.5, JP18.6, JP18.7, JP18.8
- removed net N$48: JP17.1, JP17.2, JP17.3, JP17.4, JP17.5, JP17.6, JP17.7, JP17.8
- removed net N$49: JP16.1, JP16.2, JP16.3, JP16.4, JP16.5, JP16.6, JP16.7, JP16.8
- removed net N$5: J5.1, J5.2, J5.3, J5.4, J5.5, J5.6, X1.GPIO16
- removed net N$53: LED1.C, R5.1
- removed net N$57: R7.1, SJ1.2, U2.PROG
- removed net N$60: R8.1, SJ1.1
- removed net VBAT1: C4.1, CN2.2, U2.VBAT
- removed net VDD: DC3V3.VOUT, J15.1, J15.10, J15.11, J15.2, J15.3, J15.4, J15.5, J15.6, J15.7, J15.8, J15.9, J17.1, J17.10, J17.11, J17.2, J17.3, J17.4, J17.5, J17.6, J17.7, J17.8, J17.9, JP33.1, JP33.10, JP33.11, JP33.12, JP33.2, JP33.3, JP33.4, JP33.5, JP33.6, JP33.7, JP33.8, JP33.9, JP34.1, JP34.10, JP34.11, JP34.12, JP34.2, JP34.3, JP34.4, JP34.5, JP34.6, JP34.7, JP34.8, JP34.9, U1.OUT, X1.VCC
- removed net VDD1: C3.1, LED1.A, U2.VDD, X4.VBUS
- new net 3.3V: DC3V3.VOUT, J15.1, J15.10, J15.11, J15.2, J15.3, J15.4, J15.5, J15.6, J15.7, J15.8, J15.9, J17.1, J17.10, J17.11, J17.2, J17.3, J17.4, J17.5, J17.6, J17.7, J17.8, J17.9, JP33.1, JP33.10, JP33.11, JP33.12, JP33.2, JP33.3, JP33.4, JP33.5, JP33.6, JP33.7, JP33.8, JP33.9, JP34.1, JP34.10, JP34.11, JP34.12, JP34.2, JP34.3, JP34.4, JP34.5, JP34.6, JP34.7, JP34.8, JP34.9, R1.1, R2.1, R3.1, U3.VBAT@1, U3.VBAT@2, X1.VCC
- new net N$13: SIMCARD.CLK, U3.SIM_CLK
- new net N$4: X5.GND1, X5.GND2
- new net PWD_KEY: J5.1, J5.2, J5.3, J5.4, J5.5, J5.6, U3.PWR_KEY, X1.GPIO16
- new net RESET_KEY: U3.RST
- new net UART_RX: J2.1, J2.2, J2.3, J2.4, J2.5, J2.6, U3.UART_TXD, X1.GPIO13
- new net UART_TX: J4.1, J4.2, J4.3, J4.4, J4.5, J4.6, U3.UART_RXD, X1.GPIO14
- new net V_BATT: C4.1, CN2.2, D1.A, U2.VBAT
- net GND: now also JCB_MICROUSB.GND, R4.1, SIMCARD.GND, STD_MICROUSB.GND, U3.GND, U3.GND@1, U3.GND@2, U3.GND@3, U3.GND@4, U3.GND@5, U3.GND@6, U3.GND@7, U3.GND@8, X3.GND1, X3.GND2, X3.GND3, X3.GND4; no longer C3.2, LED2.C, R8.2, U1.GND, X3.GND, X4.GND
- net N$1: now also R250.1, U3.GSM_RF; no longer J2.1, J2.2, J2.3, J2.4, J2.5, J2.6, X1.GPIO13
- net N$10: now also SIMCARD.RST, U3.SIM_RST; no longer J9.1, J9.2, J9.3, J9.4, J9.5, J9.6, X1.GPIO15
- net N$12: now also JP1.1, R3.2; no longer J11.1, J11.2, J11.3, J11.4, J11.5, J11.6
- net N$21: now also JP3.1, R1.2, X1.RESET; no longer JP1.1, JP1.2, JP1.3, JP1.4, JP1.5, JP1.6, JP1.7, JP1.8
- net N$22: now also SIMCARD.I/O, U3.SIM_DATA; no longer JP2.1, JP2.2, JP2.3, JP2.4, JP2.5, JP2.6, JP2.7, JP2.8
- net N$23: now also SIMCARD.VCC, U3.VSIM; no longer JP3.1, JP3.2, JP3.3, JP3.4, JP3.5, JP3.6, JP3.7, JP3.8
- net N$24: now also R7.1, U2.PROG; no longer JP4.1, JP4.2, JP4.3, JP4.4, JP4.5, JP4.6, JP4.7, JP4.8
- net N$3: now also R250.2, X3.ANT, X5.ANT; no longer J4.1, J4.2, J4.3, J4.4, J4.5, J4.6, X1.GPIO14
- net N$55: no longer R5.2
- net N$59: now also LED4.A; no longer LED2.A
- net N$6: now also JP2.1, R4.2, X1.GPIO15; no longer J6.1, J6.2, J6.3, J6.4, J6.5, J6.6, X1.CH_PD
- net N$7: now also X5.GND3, X5.GND4; no longer JP23.1, JP23.2, JP23.3, JP23.4, JP23.5, JP23.6, JP23.7, JP23.8
- net N$9: now also JP4.1, R2.2, X1.CH_PD; no longer J8.1, J8.2, J8.3, J8.4, J8.5, J8.6, X1.RESET
- net VCC: now also D1.C, JCB_MICROUSB.VBUS, LED4.C, STD_MICROUSB.VBUS, U2.VDD; no longer U1.EN, U1.IN, X3.VBUS
Other:
- moved on the sheet: C4, CN2, DC3V3, J1, J10, J12, J13, J14, J15, J16, J17, J18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

Commit message: More stuff
ff
Parts:
- removed DC3V3: R-78C1.8-1.0, dc-dc-converter:R-78C1.8-1.0
- removed J10: (no value), SparkFun-Connectors:M06NO_SILK_FEMALE_PTH
- removed JP1, JP2, JP4: (no value), adafruit:PINHD-1X1CB
- removed R2, R4: 10k, eagle-ltspice:R0204/7
- added C1: 1uF, microbuilder:CAP_CERAMIC0603_NO
- added C2, C3: 10µF, microbuilder:CAP_CERAMIC0805-NOOUTLINE
- added LED1: Red, adafruit:LED5MM
- added R12, R5, R9: 10k, eagle-ltspice:R0204/7
- added SW1, SW2: KMR2, microbuilder:SWITCH_TACT_SMT4.6X2.8
- added U1: (no value), microbuilder:VREG_SOT23-5
- added X2: (no value), adafruit:ANTENNA_U.FL
- D1: value 1N4148 -> MBR120; device SparkFun-DiscreteSemi:DIODE1N4148 -> microbuilder:DIODE-SCHOTTKYSOD-123
Connections:
- removed net N$11: J10.1, J10.2, J10.3, J10.4, J10.5, J10.6, X1.GPIO2
- removed net N$12: JP1.1, R3.2, X1.GPIO0
- removed net N$21: JP3.1, R1.2, X1.RESET
- removed net N$6: JP2.1, R4.2, X1.GPIO15
- removed net N$9: JP4.1, R2.2, X1.CH_PD
- new net CH_PD: R5.2, X1.CH_PD
- new net GPIO0: JP3.1, R12.2, SW2.S, SW2.S1, X1.GPIO0
- new net GPIO02: X1.GPIO2
- new net GPIO15: R9.1, X1.GPIO15
- new net GPIO2: R3.2
- new net N$5: LED1.C, R12.1
- new net RESET: R1.2, SW1.S, SW1.S1, X1.RESET
- net 3.3V: now also C1.1, C2.1, LED1.A, R5.1; no longer DC3V3.VOUT, R2.1
- net GND: now also C1.2, C2.2, C3.2, R9.2, SW1.P, SW1.P1, SW2.P, SW2.P1, X2.GND@0, X2.GND@1; no longer DC3V3.GND, R4.1
- net N$3: now also X2.SIGNAL
- net VCC: now also C3.1, U1.EN, U1.IN; no longer DC3V3.VIN
Other:
- moved on the sheet: J1, J12, J13, JP3, R1, R3
