File: xns-ip67-ESP12-Temp.sch (EAGLE design)
At the start: 76 parts, among them CN2 JSTPH, J1 DCJ0202, SW1 KMR2, SW2 KMR2, U2 MCP73831T-2ACI/OT, U3 A7, X1 ESP-12E

Commit message: New board for Temp
New board for Temp logging with A7, Power lines is routed
Parts:
- removed C1: 1uF, microbuilder:CAP_CERAMIC0603_NO
- removed C2, C3: 10µF, microbuilder:CAP_CERAMIC0805-NOOUTLINE
- removed J21, J22, J23: (no value), SparkFun-Connectors:M06NO_SILK_FEMALE_PTH
- removed JP3: (no value), adafruit:PINHD-1X1CB
- removed JP37: (no value), pinhead:PINHD-1X5
- removed LED1: Red, adafruit:LED5MM
- removed R250: (no value), eagle-ltspice:R0204/7
- removed X3: (no value), adafruit:SMACONNECTOR_EDGE
- removed X5: (no value), adafruit:SMACONNECTOR
- added C5, C6: 10uF, capacitor-wima:C2.5/2
- added C7: 1uF, capacitor-wima:C2.5/2
- added DEEPSLEEP, J11, J12, J13, J9: (no value), SparkFun-Connectors:M031X03_NO_SILK
- added J10: (no value), SparkFun-Connectors:M07NO_SILK
- added Q2: BSN20, Discrete:MOSFET-N'SOT23'
- J14: device SparkFun-Connectors:M111X11_NO_SILK -> SparkFun-Connectors:M031X03_NO_SILK
- J15, J16, J17: device SparkFun-Connectors:M111X11_NO_SILK -> SparkFun-Connectors:M07NO_SILK
- J18, J19: device SparkFun-Connectors:M06NO_SILK_FEMALE_PTH -> SparkFun-Connectors:M07NO_SILK
- J20: device SparkFun-Connectors:M06NO_SILK_FEMALE_PTH -> SparkFun-Connectors:M06FEMALE_LOCK
Connections:
- removed net N$19: J21.1, J21.2, J21.3, J21.4, J21.5, J21.6
- removed net N$20: J22.1, J22.2, J22.3, J22.4, J22.5, J22.6
- removed net N$5: LED1.C, R12.1
- removed net N$6: J7.1, J7.2, J7.3, X1.GPIO4
- removed net N$7: X5.GND3, X5.GND4
- removed net N$70: J23.1, J23.2, J23.3, J23.4, J23.5, J23.6
- removed net N$9: J8.1, J8.2, J8.3, X1.GPIO5
- removed net PWD_KEY: J2.1, J2.2, J2.3, U3.PWR_KEY, X1.GPIO16
- new net N$12: J10.1, J10.2, J10.3, J10.4, J10.5, J10.6, J10.7
- new net N$14: J15.1, J15.2, J15.3, J15.4, J15.5, J15.6, J15.7
- new net N$15: J16.1, J16.2, J16.3, J16.4, J16.5, J16.6, J16.7
- new net PWR_KEY: DEEPSLEEP.2, J2.1, J2.2, J2.3, X1.GPIO16
- net 3.3V: now also C6.1, C7.1, R12.1, U1.OUT; no longer C1.1, C2.1, J15.1, J15.10, J15.11, J15.2, J15.3, J15.4, J15.5, J15.6, J15.7, J15.8, J15.9, J17.1, J17.10, J17.11, J17.2, J17.3, J17.4, J17.5, J17.6, J17.7, J17.8, J17.9, LED1.A
- net CH_PD: now also J14.1, J14.2, J14.3
- net GND: now also C5.2, C6.2, C7.2, J20.1, Q2.S, U1.GND; no longer C1.2, C2.2, C3.2, J14.1, J14.10, J14.11, J14.2, J14.3, J14.4, J14.5, J14.6, J14.7, J14.8, J14.9, J16.1, J16.10, J16.11, J16.2, J16.3, J16.4, J16.5, J16.6, J16.7, J16.8, J16.9, JP37.1, X3.GND1, X3.GND2, X3.GND3, X3.GND4
- net GPIO0: now also J9.1, J9.2, J9.3, Q2.G; no longer JP3.1
- net GPIO15: now also J12.1, J12.2, J12.3, U3.PWR_KEY
- net GPIO2: now also J13.1, J13.2, J13.3
- net N$1: now also J3.1, J3.2, J3.3, X1.GPIO14; no longer R250.1, U3.GSM_RF
- net N$16: now also J17.1, J17.2, J17.3, J17.4, J17.5, J17.6, J17.7; no longer J18.1, J18.2, J18.3, J18.4, J18.5, J18.6
- net N$17: now also J18.1, J18.2, J18.3, J18.4, J18.5, J18.6, J18.7; no longer J19.1, J19.2, J19.3, J19.4, J19.5, J19.6
- net N$18: now also J19.1, J19.2, J19.3, J19.4, J19.5, J19.6, J19.7; no longer J20.1, J20.2, J20.3, J20.4, J20.5, J20.6
- net N$3: now also U3.GSM_RF; no longer R250.2, X3.ANT, X5.ANT
- net N$4: now also J5.1, J5.2, J5.3, X1.GPIO13; no longer X5.GND1, X5.GND2
- net RESET: now also DEEPSLEEP.3, J11.1, J11.2, J11.3
- net RESET_KEY: now also Q2.D
- net RX: now also J20.4; no longer JP37.4
- net TX: now also J20.5; no longer JP37.5
- net UART_RX: now also J7.1, J7.2, J7.3, X1.GPIO4; no longer J5.1, J5.2, J5.3, X1.GPIO13
- net UART_TX: now also J8.1, J8.2, J8.3, X1.GPIO5; no longer J3.1, J3.2, J3.3, X1.GPIO14
- net VCC: now also C5.1; no longer C3.1
Other:
- moved on the sheet: D1, J20, J4, J5, J6, J7, J8, R1, R3, R5, R9, SW1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

Commit message: Eagle Upgrade, Routing finished alpha
Parts:
- removed JCB_MICROUSB: (no value), jcbrataas-2:USB
- removed JP10, JP11, JP12, JP13, JP14, JP15, JP25, JP26, JP27, JP28, JP29, JP30, JP35, JP36: (no value), adafruit:PINHD-1X8CLEANBIG
- removed SW1, SW2: KMR2, microbuilder:SWITCH_TACT_SMT4.6X2.8
- added 5V: (no value), SparkFun-Connectors:M01NOSILK-KIT
- added DATAEXCHANGE: (no value), SparkFun-Connectors:M06FEMALE_LOCK
- added J21, J22, J23, J24, J35, J36, J37, J38, J39, J40, J41, J42, J43: (no value), SparkFun-Connectors:M08NO_SILK_FEMALE_PTH
- added PROG, RESET: KMR2, microbuilder:SWITCH_TACT_SMT4.6X2.8
- J11, J12, J13, J14, J2, J3, J4, J5, J6, J7, J8, J9: device SparkFun-Connectors:M031X03_NO_SILK -> SparkFun-Connectors:M01NOSILK-KIT
- J20: device SparkFun-Connectors:M06FEMALE_LOCK -> SparkFun-Connectors:M08NO_SILK_FEMALE_PTH
- U2: value MCP73831T-2ACI/OT -> MCP73831
Connections:
- net N$22 renamed SIM_DATA
- net N$23 renamed VSIM
- removed net N$30: JP10.1, JP10.2, JP10.3, JP10.4, JP10.5, JP10.6, JP10.7, JP10.8
- removed net N$31: JP11.1, JP11.2, JP11.3, JP11.4, JP11.5, JP11.6, JP11.7, JP11.8
- removed net N$32: JP12.1, JP12.2, JP12.3, JP12.4, JP12.5, JP12.6, JP12.7, JP12.8
- removed net N$33: JP13.1, JP13.2, JP13.3, JP13.4, JP13.5, JP13.6, JP13.7, JP13.8
- removed net N$34: JP14.1, JP14.2, JP14.3, JP14.4, JP14.5, JP14.6, JP14.7, JP14.8
- removed net N$35: JP15.1, JP15.2, JP15.3, JP15.4, JP15.5, JP15.6, JP15.7, JP15.8
- removed net N$36: JP30.1, JP30.2, JP30.3, JP30.4, JP30.5, JP30.6, JP30.7, JP30.8
- removed net N$37: JP29.1, JP29.2, JP29.3, JP29.4, JP29.5, JP29.6, JP29.7, JP29.8
- removed net N$38: JP28.1, JP28.2, JP28.3, JP28.4, JP28.5, JP28.6, JP28.7, JP28.8
- removed net N$39: JP27.1, JP27.2, JP27.3, JP27.4, JP27.5, JP27.6, JP27.7, JP27.8
- removed net N$40: JP26.1, JP26.2, JP26.3, JP26.4, JP26.5, JP26.6, JP26.7, JP26.8
- removed net N$41: JP25.1, JP25.2, JP25.3, JP25.4, JP25.5, JP25.6, JP25.7, JP25.8
- removed net N$50: JP35.1, JP35.2, JP35.3, JP35.4, JP35.5, JP35.6, JP35.7, JP35.8
- removed net N$51: JP36.1, JP36.2, JP36.3, JP36.4, JP36.5, JP36.6, JP36.7, JP36.8
- removed net PWR_KEY: DEEPSLEEP.2, J2.1, J2.2, J2.3, X1.GPIO16
- new net ADC: J8.1, X1.ADC
- new net GPIO12: J13.1, X1.GPIO12
- new net GPIO13: J14.1, X1.GPIO13
- new net GPIO14: J12.1, X1.GPIO14
- new net GPIO16: DEEPSLEEP.2, J11.1, X1.GPIO16
- new net N$11: J40.1, J40.2, J40.3, J40.4, J40.5, J40.6, J40.7, J40.8
- new net N$19: J42.1, J42.2, J42.3, J42.4, J42.5, J42.6, J42.7, J42.8
- new net N$20: J36.1, J36.2, J36.3, J36.4, J36.5, J36.6, J36.7, J36.8
- new net N$21: J43.1, J43.2, J43.3, J43.4, J43.5, J43.6, J43.7, J43.8
- new net N$5: J23.1, J23.2, J23.3, J23.4, J23.5, J23.6, J23.7, J23.8
- new net N$6: J24.1, J24.2, J24.3, J24.4, J24.5, J24.6, J24.7, J24.8
- new net N$7: J35.1, J35.2, J35.3, J35.4, J35.5, J35.6, J35.7, J35.8
- new net N$9: J38.1, J38.2, J38.3, J38.4, J38.5, J38.6, J38.7, J38.8
- new net SIM_CLK: SIMCARD.RST, U3.SIM_CLK
- new net SIM_RST: SIMCARD.CLK, U3.SIM_RST
- net CH_PD: now also J9.1; no longer J14.1, J14.2, J14.3
- net GND: now also DATAEXCHANGE.1, PROG.P, PROG.P1, RESET.P, RESET.P1; no longer J20.1, JCB_MICROUSB.GND, SW1.P, SW1.P1, SW2.P, SW2.P1
- net GPIO0: now also J4.1, PROG.S, PROG.S1; no longer J9.1, J9.2, J9.3, SW2.S, SW2.S1
- net GPIO15: now also J6.1; no longer J12.1, J12.2, J12.3
- net GPIO2: now also J5.1; no longer J13.1, J13.2, J13.3
- net N$1: now also J20.1, J20.2, J20.3, J20.4, J20.5, J20.6, J20.7, J20.8; no longer J3.1, J3.2, J3.3, X1.GPIO14
- net N$10: now also J39.1, J39.2, J39.3, J39.4, J39.5, J39.6, J39.7, J39.8; no longer SIMCARD.RST, U3.SIM_RST
- net N$13: now also J41.1, J41.2, J41.3, J41.4, J41.5, J41.6, J41.7, J41.8; no longer SIMCARD.CLK, U3.SIM_CLK
- net N$2: now also J21.1, J21.2, J21.3, J21.4, J21.5, J21.6, J21.7, J21.8; no longer J4.1, J4.2, J4.3, X1.GPIO12
- net N$4: now also J22.1, J22.2, J22.3, J22.4, J22.5, J22.6, J22.7, J22.8; no longer J5.1, J5.2, J5.3, X1.GPIO13
- net N$8: now also J37.1, J37.2, J37.3, J37.4, J37.5, J37.6, J37.7, J37.8; no longer J6.1, J6.2, J6.3, X1.ADC
- net RESET: now also J7.1, RESET.S, RESET.S1; no longer J11.1, J11.2, J11.3, SW1.S, SW1.S1
- net RX: now also DATAEXCHANGE.4, J3.1; no longer J20.4
- net TX: now also DATAEXCHANGE.5, J2.1; no longer J20.5
- net UART_RX: no longer J7.1, J7.2, J7.3
- net UART_TX: no longer J8.1, J8.2, J8.3
- net VCC: now also 5V.1; no longer JCB_MICROUSB.VBUS
Other:
- note added: "ESP8266"
- note added: "External Power Connector"
- note added: "External Power Source"
- note added: "GPRS, GPS, SIM CARD"
- note added: "LiPo Charging"
- note added: "Power and Filter"
- moved on the sheet: C4, C5, C6, C7, CN2, D1, DEEPSLEEP, J1, J10, J15, J16, J17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

Commit message: Cleanup, add PIN's
Added Pin for GPIO’s
Parts:
- added J44, J45: (no value), SparkFun-Connectors:M01NOSILK-KIT
Connections:
- net UART_RX: now also J45.1
- net UART_TX: now also J44.1
Changed lines of the file:
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@@
 <part name="5V" library="SparkFun-Connectors" deviceset="M01" device="NOSILK-KIT"/>
 <part name="P+2" library="supply1" deviceset="VCC" device=""/>
+<part name="J44" library="SparkFun-Connectors" deviceset="M01" device="NOSILK-KIT"/>
+<part name="J45" library="SparkFun-Connectors" deviceset="M01" device="NOSILK-KIT"/>
 </parts>
 <sheets>
@@
 <attribute name="VALUE" x="166.37" y="198.12" size="1.778" layer="96" rot="R90"/>
 </instance>
+<instance part="J44" gate="G$1" x="62.23" y="182.88" rot="R270"/>
+<instance part="J45" gate="G$1" x="71.12" y="182.88" rot="R270"/>
 </instances>
 <busses>
@@
 <label x="49.53" y="149.86" size="1.778" layer="95"/>
 </segment>
+<segment>
+<pinref part="J45" gate="G$1" pin="1"/>
+<wire x1="71.12" y1="175.26" x2="71.12" y2="170.18" width="0.1524" layer="91"/>
+<label x="71.12" y="166.37" size="1.778" layer="95" rot="R90"/>
+</segment>
 </net>
 <net name="UART_TX" class="0">
@@
 <label x="49.53" y="152.4" size="1.778" layer="95"/>
 </segment>
+<segment>
+<pinref part="J44" gate="G$1" pin="1"/>
+<wire x1="62.23" y1="175.26" x2="62.23" y2="170.18" width="0.1524" layer="91"/>
+<label x="62.23" y="166.37" size="1.778" layer="95" rot="R90"/>
+</segment>
 </net>
